File: AK Flex Buttons/AK Flex Buttons.kicad_sch (KiCad schematic)
At the start: 0 parts

Commit message: Added more findings
Parts:
- added C1: C, symbol Device:C
- added SW1: SW_Push, symbol Switch:SW_Push
Connections:
- new net GND: C1.2, SW1.1
- new net REV: C1.1, SW1.2
